File: weather-station.kicad_sch (KiCad schematic)
At the start: 4 parts, among them U1 ESP32-WROOM-32, U2 BME280

Commit message: Added PCB after schematics, warnings yet to be resolved
Parts:
- added U3: ER_OLEDM0.91_1x-I2C, Display:ER_OLEDM0.91_1x-I2C, symbol Display_Graphic:ER_OLEDM0.91_1x-I2C
- R1, R2: footprint (none) -> Resistor_SMD:R_1206_3216Metric_Pad1.30x1.75mm_HandSolder
Connections:
- net +3V3: now also U3.2 (VCC)
- net GND: now also U3.1 (GND)
- net at R2.2, U1.33 (IO21), U2.3 (SDI): now also U3.4 (SDA)
- net at R1.2, U1.36 (IO22), U2.4 (SCK): now also U3.3 (SCL)
